Commit message: 12

File: smart_conveyor/smart_conv.urdf (robot description, URDF)
Before this commit: robot Smart_Conveyor, 5 links, 4 joints
Links:
- link Link_1: geometry collision mesh filename=/home/apshirazi/Isaac_sim_ws/smart_conveyor/collision/Belt_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 scale=0.001 0.001 0.001; visual mesh filename=/home/apshirazi/Isaac_sim_ws/smart_conveyor/Belt_Base.stl scale=0.001 0.001 0.001
- link Link_2: geometry collision mesh filename=/home/apshirazi/Isaac_sim_ws/smart_conveyor/collision/Belt_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 scale=0.001 0.001 0.001; visual mesh filename=/home/apshirazi/Isaac_sim_ws/smart_conveyor/Belt_Surface.stl scale=0.001 0.001 0.001
- link base_link: geometry collision mesh filename=/home/apshirazi/Isaac_sim_ws/smart_conveyor/collision/Conv_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 scale=0.001 0.001 0.001; visual mesh filename=/home/apshirazi/Isaac_sim_ws/smart_conveyor/Conv_Base.stl scale=0.001 0.001 0.001
- link track_link: geometry collision mesh filename=/home/apshirazi/Isaac_sim_ws/smart_conveyor/collision/Robot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 scale=0.001 0.001 0.001; visual mesh filename=/home/apshirazi/Isaac_sim_ws/smart_conveyor/Robotic_Track.s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 scale=0.001 0.001 0.001
Joints:
- joint Joint_1: limit lower=0 upper=20 effort=100 velocity=10 -> lower=0 upper=4.55 effort=100 velocity=10
- joint Joint_2: limit lower=0 upper=20 effort=100 velocity=10 -> lower=0 upper=0.5 effort=100 velocity=10
- joint rob_to_box: origin xyz=0 0 0.2 rpy=1.57 0 0 -> xyz=0 0 0.2 rpy=1.57 0 1.57

Commit message: 12

File: smart_conveyor/smart_conv.urdf (robot description, URDF)
Before this commit: robot Smart_Conveyor, 5 links, 4 joints
Joints:
- joint rob_to_box: origin xyz=0 0 0.2 rpy=1.57 0 1.57 -> xyz=0 0 0.2 rpy=1.57 0 0
