Commit message: 2ROB

File: robot_2/IRB6620_R2_ROS.urdf (robot description, URDF)
Before this commit: robot IRB6620_R2, 14 links, 13 joints
Joints:
- joint Joint_1: origin xyz=0 0 0.2135 rpy=0 0 0 -> xyz=0 0 0.2135 rpy=0 0 3.14159

Commit message: Works

File: robot_2/IRB6620_R2_ROS.urdf (robot description, URDF)
Before this commit: robot IRB6620_R2, 14 links, 13 joints
Joints:
- joint Joint_1: limit lower=-2.967 upper=2.967 effort=10000 velocity=1.745 -> lower=-2.967 upper=2.967 effort=0 velocity=1.745
- joint Joint_2: limit lower=-1.134 upper=1.134 effort=10000 velocity=1.57 -> lower=-1.134 upper=1.134 effort=0 velocity=1.57
- joint Joint_3: limit lower=-3.141 upper=1.221 effort=10000 velocity=1.57 -> lower=-3.141 upper=1.221 effort=0 velocity=1.57
- joint Joint_4: limit lower=-5.235 upper=5.235 effort=10000 velocity=2.617 -> lower=-5.235 upper=5.235 effort=0 velocity=2.617
- joint Joint_5: limit lower=-2.268 upper=2.268 effort=10000 velocity=2.095 -> lower=-2.268 upper=2.268 effort=0 velocity=2.095
- joint Joint_6: limit lower=-5.235 upper=5.235 effort=10000 velocity=3.316 -> lower=-5.235 upper=5.235 effort=0 velocity=3.316
- joint Joint_8: limit lower=0 upper=1.57 effort=10000 velocity=10.0 -> lower=0 upper=1.57 effort=0 velocity=10.0

Commit message: All Done

File: robot_2/IRB6620_R2_ROS.urdf (robot description, URDF)
Before this commit: robot IRB6620_R2, 14 links, 13 joints
Joints:
- joint Joint_8: axis 1 0 0 -> (none); limit lower=0 upper=1.57 effort=0 velocity=10.0 -> (none); type revolute -> fixed

Commit message: Nailing Got Better

File: robot_2/IRB6620_R2_ROS.urdf (robot description, URDF)
Before this commit: robot IRB6620_R2, 14 links, 13 joints
Joints:
- joint Link_6-tool1: origin xyz=0.352827674 -0.31656238 0.0519 rpy=0 -1.57079632679 0 -> xyz=0.391037674 -0.34051238 0.00172 rpy=0 -1.57079632679 0
