Commit message: TCPs Fixed, Start The Strategy Test

File: robot/IRB6620_R1_ROS.urdf (robot description, URDF)
Before this commit: robot IRB6620_R1, 16 links, 15 joints
Joints:
- joint Link_6-tool0: origin xyz=0.087264505 0.2964 -0.24 rpy=0 0 0 -> xyz=0.087264505 0.0 -0.24 rpy=-3.1415927 0 0

File: robot_2/IRB6620_R2_ROS.urdf (robot description, URDF)
Before this commit: robot IRB6620_R2, 14 links, 13 joints
Joints:
- joint Link_6-tool0: origin xyz=0.618323344138 0.455185395 -0.05935 rpy=0 -1.57079632679 0 -> xyz=0.618323344138 0.155185395 -0.11003 rpy=0.0 1.57079632679 0.0

Commit message: Effort Fixed

File: robot/IRB6620_R1_ROS.urdf (robot description, URDF)
Before this commit: robot IRB6620_R1, 16 links, 15 joints
Joints:
- joint Joint_1: limit lower=-2.967 upper=2.967 effort=0 velocity=1.745 -> lower=-2.967 upper=2.967 effort=10000 velocity=1.745
- joint Joint_2: limit lower=-1.134 upper=1.134 effort=0 velocity=1.57 -> lower=-1.134 upper=1.134 effort=10000 velocity=1.57
- joint Joint_3: limit lower=-3.141 upper=1.221 effort=0 velocity=1.57 -> lower=-3.141 upper=1.221 effort=10000 velocity=1.57
- joint Joint_4: limit lower=-5.235 upper=5.235 effort=0 velocity=2.617 -> lower=-5.235 upper=5.235 effort=10000 velocity=2.617
- joint Joint_5: limit lower=-2.268 upper=2.268 effort=0 velocity=2.095 -> lower=-2.268 upper=2.268 effort=10000 velocity=2.095
- joint Joint_6: limit lower=-5.235 upper=5.235 effort=0 velocity=3.316 -> lower=-5.235 upper=5.235 effort=10000 velocity=3.316
- joint Joint_8: limit lower=0 upper=1.57 effort=0 velocity=10.0 -> lower=0 upper=1.57 effort=10000 velocity=10.0

File: robot_2/IRB6620_R2_ROS.urdf (robot description, URDF)
Before this commit: robot IRB6620_R2, 14 links, 13 joints
Joints:
- joint Joint_1: limit lower=-2.967 upper=2.967 effort=0 velocity=1.745 -> lower=-2.967 upper=2.967 effort=10000 velocity=1.745
- joint Joint_2: limit lower=-1.134 upper=1.134 effort=0 velocity=1.57 -> lower=-1.134 upper=1.134 effort=10000 velocity=1.57
- joint Joint_3: limit lower=-3.141 upper=1.221 effort=0 velocity=1.57 -> lower=-3.141 upper=1.221 effort=10000 velocity=1.57
- joint Joint_4: limit lower=-5.235 upper=5.235 effort=0 velocity=2.617 -> lower=-5.235 upper=5.235 effort=10000 velocity=2.617
- joint Joint_5: limit lower=-2.268 upper=2.268 effort=0 velocity=2.095 -> lower=-2.268 upper=2.268 effort=10000 velocity=2.095
- joint Joint_6: limit lower=-5.235 upper=5.235 effort=0 velocity=3.316 -> lower=-5.235 upper=5.235 effort=10000 velocity=3.316
- joint Joint_8: limit lower=0 upper=1.57 effort=0 velocity=10.0 -> lower=0 upper=1.57 effort=10000 velocity=10.0

Commit message: Home Pose Fixed, Both Robots Working

File: robot/IRB6620_R1_ROS.urdf (robot description, URDF)
Before this commit: robot IRB6620_R1, 16 links, 15 joints
Joints:
- joint Joint_8: axis 1 0 0 -> (none); limit lower=0 upper=1.57 effort=10000 velocity=10.0 -> (none); type revolute -> fixed

Commit message: Conveyor Shaking Might be Fixed

File: robot/IRB6620_R1_ROS.urdf (robot description, URDF)
Before this commit: robot IRB6620_R1, 16 links, 15 joints
Joints:
- joint Link_6-tool0: origin xyz=0.087264505 0.0 -0.24 rpy=-3.1415927 0 0 -> xyz=0.087264505 0.0053 -0.24 rpy=-3.1415927 0 0

Commit message: Efforts Fixed

File: robot/IRB6620_R1_ROS.urdf (robot description, URDF)
Before this commit: robot IRB6620_R1, 16 links, 15 joints
Joints:
- joint Joint_1: limit lower=-2.967 upper=2.967 effort=10000 velocity=1.745 -> lower=-2.967 upper=2.967 effort=100 velocity=1.745
- joint Joint_2: limit lower=-1.134 upper=1.134 effort=10000 velocity=1.57 -> lower=-1.134 upper=1.134 effort=100 velocity=1.57
- joint Joint_3: limit lower=-3.141 upper=1.221 effort=10000 velocity=1.57 -> lower=-3.141 upper=1.221 effort=100 velocity=1.57
- joint Joint_4: limit lower=-5.235 upper=5.235 effort=10000 velocity=2.617 -> lower=-5.235 upper=5.235 effort=100 velocity=2.617
- joint Joint_5: limit lower=-2.268 upper=2.268 effort=10000 velocity=2.095 -> lower=-2.268 upper=2.268 effort=100 velocity=2.095
- joint Joint_6: limit lower=-5.235 upper=5.235 effort=10000 velocity=3.316 -> lower=-5.235 upper=5.235 effort=100 velocity=3.316

File: robot_2/IRB6620_R2_ROS.urdf (robot description, URDF)
Before this commit: robot IRB6620_R2, 14 links, 13 joints
Joints:
- joint Joint_1: limit lower=-2.967 upper=2.967 effort=0 velocity=1.745 -> lower=-2.967 upper=2.967 effort=100 velocity=1.745
- joint Joint_2: limit lower=-1.134 upper=1.134 effort=0 velocity=1.57 -> lower=-1.134 upper=1.134 effort=100 velocity=1.57
- joint Joint_4: limit lower=-5.235 upper=5.235 effort=0 velocity=2.617 -> lower=-5.235 upper=5.235 effort=100 velocity=2.617
- joint Joint_5: limit lower=-2.268 upper=2.268 effort=0 velocity=2.095 -> lower=-2.268 upper=2.268 effort=100 velocity=2.095
- joint Joint_6: limit lower=-5.235 upper=5.235 effort=0 velocity=3.316 -> lower=-5.235 upper=5.235 effort=100 velocity=3.316

Commit message: Damping Stiffness Values Added

File: robot/IRB6620_R1_ROS.urdf (robot description, URDF)
Before this commit: robot IRB6620_R1, 16 links, 15 joints
Joints:
- joint Joint_1: limit lower=-2.967 upper=2.967 effort=100 velocity=1.745 -> lower=-2.967 upper=2.967 effort=10000 velocity=1.745
- joint Joint_2: limit lower=-1.134 upper=1.134 effort=100 velocity=1.57 -> lower=-1.134 upper=1.134 effort=10000 velocity=1.57
- joint Joint_3: limit lower=-3.141 upper=1.221 effort=100 velocity=1.57 -> lower=-3.141 upper=1.221 effort=10000 velocity=1.57
- joint Joint_4: limit lower=-5.235 upper=5.235 effort=100 velocity=2.617 -> lower=-5.235 upper=5.235 effort=10000 velocity=2.617
- joint Joint_5: limit lower=-2.268 upper=2.268 effort=100 velocity=2.095 -> lower=-2.268 upper=2.268 effort=10000 velocity=2.095
- joint Joint_6: limit lower=-5.235 upper=5.235 effort=100 velocity=3.316 -> lower=-5.235 upper=5.235 effort=10000 velocity=3.316

File: robot_2/IRB6620_R2_ROS.urdf (robot description, URDF)
Before this commit: robot IRB6620_R2, 14 links, 13 joints
Joints:
- joint Joint_1: limit lower=-2.967 upper=2.967 effort=100 velocity=1.745 -> lower=-2.967 upper=2.967 effort=10000 velocity=1.745
- joint Joint_2: limit lower=-1.134 upper=1.134 effort=100 velocity=1.57 -> lower=-1.134 upper=1.134 effort=10000 velocity=1.57
- joint Joint_3: limit lower=-3.141 upper=1.221 effort=0 velocity=1.57 -> lower=-3.141 upper=1.221 effort=10000 velocity=1.57
- joint Joint_4: limit lower=-5.235 upper=5.235 effort=100 velocity=2.617 -> lower=-5.235 upper=5.235 effort=10000 velocity=2.617
- joint Joint_5: limit lower=-2.268 upper=2.268 effort=100 velocity=2.095 -> lower=-2.268 upper=2.268 effort=10000 velocity=2.095
- joint Joint_6: limit lower=-5.235 upper=5.235 effort=100 velocity=3.316 -> lower=-5.235 upper=5.235 effort=10000 velocity=3.316

Commit message: 12

File: robot/IRB6620_R1_ROS.urdf (robot description, URDF)
Before this commit: robot IRB6620_R1, 16 links, 15 joints
Joints:
- joint Link_6-tool3: origin xyz=0.226962 -0.705 0.002537 rpy=-1.57079632679 0.174533 0 -> xyz=0.226962 -0.705 0.002537 rpy=-1.57079632679 0 0
